File: Hardware/v1_20230725/Design Folder/_HW_HotPlate/_HW_HotPlate.kicad_sch (KiCad schematic)
At the start: 0 parts

Commit message: Schematic library has been updated
Other:
- added sheet PWR SEQUENCE ([13] - PWR SEQUENCE.kicad_sch)
- added sheet REVISION HISTORY ([14] - REVISION HISTORY.kicad_sch)
- sheet MECHANICAL PARTS: file [08] - MECHANICAL PARTS.kicad_sch -> [12] - MECHANICAL PARTS.kicad_sch
- note added: "${COMMENT2}"
- note added: "1- Go to View -> Pge Preview Setting 2- Set Parameters based on the following Info COMMENT 1: Project Version COMMENT 2: Document Status COMMENT 3: Doc. Approval Eng. COMMENT 4: BOM Ref. DOC. COMMENT 5: PCB Ref. DOC. COMMENT 6: GBR Ref. DOC. COMMENT 7: ASM Ref. DOC. COMMENT 8: Variant Name COMMENT 9: Revision Description"
- note added: "21"
- note added: "22"
- note added: "23"
- note added: "24"
- note added: "25"
- note added: "26"
- note added: "27"
- note added: "28"
- note added: "29"
- note added: "30"
- note added: "3D Preview BOTTOM"
- note added: "3D Preview TOP"
- note added: "Board Statistics Stackup Info"
- note added: "FAN DRIVER"
- note added: "ISOLATED TRIAC DRIVER"
- note added: "LEDS DRIVER"
- note added: "MECHANICAL PARTS"
- note added: "MICROCONTROLLER"
- note added: "PCD8544 DRIVER"
- note added: "POWER SUPPLY"
- note added: "ROTARY ENCODER _ PB DRIVER"
- note added: "SHOULD BE ADDED AFTER RELEASE"
- note added: "THERMOCOUPLE DRIVER"
- note added: "USB DRIVER"
- note removed: "1- Go to View -> Pge Preview Setting 2- Set Parameters based on the following Info COMMENT 1: Project Version COMMENT 2: Document Version COMMENT 3: Doc. Approval Eng. COMMENT 4: BOM Ref. DOC. COMMENT 5: PCB Ref. DOC. COMMENT 6: GBR Ref. DOC. COMMENT 7: ASM Ref. DOC. COMMENT 8: Variant Name COMMENT 9: Revision Description"
- note removed: "DESIGN CONSIDERATION"
- note removed: "RELEASED"
