File: Hardware/v1_20230725/Design Folder/_HW_HotPlate/[03] - MCU.kicad_sch (KiCad schematic)
At the start: 21 parts, among them J301 MHDR_4POS_2.54MM_RA, U301 PIC18F24J50-I/ML, U302 SN74LVC1G17DBVR, U303 SN74LVC1G17DBVR, X301 16MHz/10ppm

Commit message: Schematic library has been updated
Other:
- note removed: "CHECKED"
- moved on the sheet: C301, C302, C303, C304, C305, C306, C307, C308, C309, C310, C311, D301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

Commit message: components have been updated
Parts:
- C301, C302: value 12pF/50V -> 12pF_50V_C0G; symbol _SCHLIB_HotPlate:CAP_12pF/50V_C0201 -> _SCHLIB_HotPlate:CAP_12pF_50V_C0G_C0201; Manufacturer (none) -> YAGEO; PCB CHECk (none) -> PCB (N/A); Part Number CC0201JRNPO9BN120 -> (none); Part Number (Manufacturer) (none) -> CC0201JRNPO9BN120; Part Number (Vendor) (none) -> 311-1585-2-ND; SCH CHECK CHECKED -> SCH (N/A); Vendor (none) -> Digikey
- C303, C304, C306, C308, C309, C311: value 100nF/6V3 -> 100nF_6V3_X7R; symbol _SCHLIB_HotPlate:CAP_100nF/6V3_C0201 -> _SCHLIB_HotPlate:CAP_100nF_6V3_X7R_C0201; Manufacturer (none) -> YAGEO; PCB CHECk (none) -> PCB (N/A); Part Number CC0201KRX7R5BB104 -> (none); Part Number (Manufacturer) (none) -> CC0201KRX7R5BB104; Part Number (Vendor) (none) -> 13-CC0201KRX7R5BB104TR-ND; SCH CHECK CHECKED -> SCH (N/A); Vendor (none) -> Digikey
- C305, C307, C310: value 10uF/16V -> 10uF_16V_X5R; symbol _SCHLIB_HotPlate:CAP_10uF/16V-C0603 -> _SCHLIB_HotPlate:CAP_10uF_16V_X5R_C0603; Manufacturer (none) -> Murata Electronics; PCB CHECk (none) -> PCB (N/A); Part Number GRT188R61C106KE13J -> (none); Part Number (Manufacturer) (none) -> GRT188R61C106KE13J; Part Number (Vendor) (none) -> 490-GRT188R61C106KE13JTR-ND; SCH CHECK CHECKED -> SCH (N/A); Vendor (none) -> Digikey
- D301: value SMF3.3 -> SMF3.3_3.3V_30A; symbol _SCHLIB_HotPlate:TVS_SMF3.3_SOD_123F -> _SCHLIB_HotPlate:DIODE_TVS_SMF3.3_3.3V_3.4V_30A(10/1000us)_SOD_123F; Ipp 30A (10/1000uS) -> (none); Manufacturer (none) -> Littelfuse Inc.; PCB CHECk (none) -> PCB (N/A); Package (none) -> SOD-123F; Part Number SMF3.3 -> (none); Part Number (Manufacturer) (none) -> SMF3.3; Part Number (Vendor) (none) -> F7701TR-ND; SCH CHECK CHECKED -> SCH (N/A); Vbr 3.4 (Vbr) -> (none); Vc 6.8 (Vc) -> (none); Vendor (none) -> Digikey
- J301: value MHDR_4POS_2.54MM_RA -> MHDR_4X1_RA_2.54MM; symbol _SCHLIB_HotPlate:CONN_MHDR_4POS_2.54MM_RA -> _SCHLIB_HotPlate:CONN_MHDR_4POS_RA_2.54MM; Manufacturer (none) -> Adam Tech; PCB CHECk (none) -> PCB (N/A); Package (none) -> THD_RA; Part Number PH1RB-04-UA -> (none); Part Number (Manufacturer) (none) -> PH1RB-04-UA; Part Number (Vendor) (none) -> 2057-PH1RB-04-UA-ND; SCH CHECK CHECKED -> SCH (N/A); Vendor (none) -> Digikey
- LED301: value RED -> RED_2V_0.02A; symbol _SCHLIB_HotPlate:LED_RED_0402 -> _SCHLIB_HotPlate:DIODE_LED_RED_2V_0.02A_632nm_LED0402; Manufacturer (none) -> Harvatek Corporation; PCB CHECk (none) -> PCB (N/A); Part Number B2841USD-20D001014U1930 -> (none); Part Number (Manufacturer) (none) -> B2841USD-20D001014U1930; Part Number (Vendor) (none) -> 3147-B2841USD-20D001014U1930TR-ND; SCH CHECK CHECKED -> SCH (N/A); VOLTAGE RATED 2V -> (none); Vendor (none) -> Digikey
- R301: value 49R9_1/20W -> 49R9_1/20W_1%; symbol _SCHLIB_HotPlate:RES_49R9_1/20W-R0201 -> _SCHLIB_HotPlate:RES_49R9_1/20W_1%_R0201; Manufacturer (none) -> Stackpole Electronics Inc; PCB CHECk (none) -> PCB (N/A); Part Number RMCF0201FT49R9 -> (none); Part Number (Manufacturer) (none) -> RMCF0201FT49R9; Part Number (Vendor) (none) -> RMCF0201FT49R9TR-ND; SCH CHECK CHECKED -> SCH (N/A); Vendor (none) -> Digikey
- R302: value 10KR_1/20W -> 10KR_1/20W_1%; symbol _SCHLIB_HotPlate:RES_10KR_1/20W-R0201 -> _SCHLIB_HotPlate:RES_10KR_1/20W_1%_R0201; Manufacturer (none) -> Stackpole Electronics Inc; PCB CHECk (none) -> PCB (N/A); Part Number RMCF0201FT10K0 -> (none); Part Number (Manufacturer) (none) -> RMCF0201FT10K0; Part Number (Vendor) (none) -> RMCF0201FT10K0TR-ND; SCH CHECK CHECKED -> SCH (N/A); Vendor (none) -> Digikey
- R303: value 100R_1/20W -> 100R_1/20W_1%; symbol _SCHLIB_HotPlate:RES_100R_1/20W-R0201 -> _SCHLIB_HotPlate:RES_100R_1/20W_1%_R0201; Manufacturer (none) -> Stackpole Electronics Inc; PCB CHECk (none) -> PCB (N/A); Part Number RMCF0201FT100R -> (none); Part Number (Manufacturer) (none) -> RMCF0201FT100R; Part Number (Vendor) (none) -> RMCF0201FT100RTR-ND; SCH CHECK CHECKED -> SCH (N/A); Vendor (none) -> Digikey
- U301: symbol _SCHLIB_HotPlate:MCU_PIC18F24J50-I/ML -> _SCHLIB_HotPlate:IC_MCU_PIC18F24J50-I/ML_8-bit_48MHz_3.6V_28-QFN (6x6); Manufacturer (none) -> Microchip Technology; PCB CHECk (none) -> PCB (N/A); Package (none) -> 28-QFN (6x6); Part Number PIC18F24J50-I/ML -> (none); Part Number (Manufacturer) (none) -> PIC18F24J50-I/ML; Part Number (Vendor) (none) -> PIC18F24J50-I/ML-ND; SCH CHECK CHECKED -> SCH (N/A); Vendor (none) -> Digikey
- U302, U303: symbol _SCHLIB_HotPlate:BUF_SN74LVC1G17DBVR_SOT-23-5 -> _SCHLIB_HotPlate:IC_BUFFER_SN74LVC1G17DBVR_NON-INV_5.5V_32mA_SOT-23-5; Manufacturer (none) -> Texas Instruments; PCB CHECk (none) -> PCB (N/A); Package (none) -> SOT-23-5; Part Number SN74LVC1G17DBVR -> (none); Part Number (Manufacturer) (none) -> SN74LVC1G17DBVR; Part Number (Vendor) (none) -> 296-11933-2-ND; SCH CHECK CHECKED -> SCH (N/A); Vendor (none) -> Digikey
- X301: value 16MHz/10ppm -> 16MHz_10ppm_12pF; symbol _SCHLIB_HotPlate:XTAL_ECS-160-12-37B-CTN-TR -> _SCHLIB_HotPlate:XTAL_ECS-160-12-37B-CTN-TR_16MHz_10ppm_12pF_4SMD-2016; Manufacturer (none) -> ECS Inc.; PCB CHECk (none) -> PCB (N/A); Part Number ECS-160-12-37B-CTN-TR -> (none); Part Number (Manufacturer) (none) -> ECS-160-12-37B-CTN-TR; Part Number (Vendor) (none) -> XC3061TR-ND; SCH CHECK CHECKED -> SCH (N/A); Vendor (none) -> Digikey
Other:
- moved on the sheet: C301, C302, C303, C304, C305, C306, C307, C308, C309, C310, C311, D301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

Commit message: Updating hardware format structure
Other:
- note added: "1: The on-chip voltage regulator is only available on parts designated with an “F”, such as PIC18F25J50. The on-chip regulator is disabled on devices with “LF” in their part number. 2: The VDDCORE/VCAP pin must never be left floating. On “F” devices, it must be connected to a capacitor, of size, CEFC, to ground. On “LF” devices, VDDCORE/VCAP must be connected to a power supply source between 2.0V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"
- note added: "DESIGN NOTE:"
- note removed: "DESIGN NOTE: 1: The on-chip voltage regulator is only available on parts designated with an “F”, such as PIC18F25J50. The on-chip regulator is disabled on devices with “LF” in their part number. 2: The VDDCORE/VCAP pin must never be left floating. On “F” devices, it must be connected to a capacitor, of size, CEFC, to ground. On “LF” devices, VDDCORE/VCAP must be connected to a power supply source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"
Changed lines of the file:
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@@
     (stroke (width 0) (type default))
   )
-  (rectangle (start 116.84 245.11) (end 170.18 281.94)
+  (rectangle (start 116.84 245.11) (end 175.26 281.94)
     (stroke (width 0) (type default))
     (fill (type none))
   )
-  (rectangle (start 119.38 247.65) (end 167.64 279.4)
+  (rectangle (start 119.38 247.65) (end 172.72 279.4)
     (stroke (width 0) (type default))
     (fill (type none))
@@
     (fill (type none))
   )
-  (rectangle (start 118.11 246.38) (end 168.91 280.67)
+  (rectangle (start 118.11 246.38) (end 173.99 280.67)
     (stroke (width 0) (type default))
     (fill (type none))
@@
     (effects (font (size 1.27 1.27)) (justify left bottom))
   )
-  (text "DESIGN NOTE:\n\n 1: The on-chip voltage regulator is only\navailable on parts designated with an “F”,\nsuch as PIC18F25J50. The on-chip\nregulator is disabled on devices with “LF”\nin their part number.\n 2: The VDDCORE/VCAP pin must never be left\nfloating. On “F” devices, it must be connected \nto a capacitor, of size, CEFC, to\nground. On “LF” devices, VDDCORE/VCAP\nmust be connected to a power supply\nsource between 2.0V and 2.7V."
+  (text "DESIGN NOTE:" (at 121.92 252.73 0)
+    (effects (font (size 1.8 1.8) bold) (justify left bottom))
+  )
+  (text " 1: The on-chip voltage regulator is only\navailable on parts designated with an “F”,\nsuch as PIC18F25J50. The on-chip\nregulator is disabled on devices with “LF”\nin their part number.\n 2: The VDDCORE/VCAP pin must never be left\nfloating. On “F” devices, it must be connected \nto a capacitor, of size, CEFC, to\nground. On “LF” devices, VDDCORE/VCAP\nmust be connected to a power supply\nsource between 2.0V and 2.7V."
     (at 121.92 276.86 0)
     (effects (font (size 1.27 1.27)) (justify left bottom))
