File: Hardware/v1_20230725/Design Folder/_HW_HotPlate/[03] - MCU.kicad_sch (KiCad schematic)
At the start: 21 parts, among them J301 MHDR_4X1_RA_2.54MM, U301 PIC18F24J50-I/ML, U302 SN74LVC1G17DBVR, U303 SN74LVC1G17DBVR, X301 16MHz_10ppm_12pF

Commit message: Library updated
Parts:
- C301, C302: symbol _SCHLIB_HotPlate:CAP_12pF_50V_C0G_C0201 -> _SCHLIB_HotPlate:CAP_CER_12pF_50V_C0G_C0201
- C303, C304, C306, C308, C309, C311: symbol _SCHLIB_HotPlate:CAP_100nF_6V3_X7R_C0201 -> _SCHLIB_HotPlate:CAP_CER_100nF_6V3_X7R_C0201
- C305, C307, C310: symbol _SCHLIB_HotPlate:CAP_10uF_16V_X5R_C0603 -> _SCHLIB_HotPlate:CAP_CER_10uF_16V_X5R_C0603
Changed lines of the file:
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@@
     )
   )
-  (symbol (lib_id "_SCHLIB_HotPlate:CAP_12pF_50V_C0G_C0201") (at 125.73 166.37 180) (unit 1)
+  (symbol (lib_id "_SCHLIB_HotPlate:CAP_CER_12pF_50V_C0G_C0201") (at 125.73 166.37 180) (unit 1)
     (in_bom yes) (on_board yes) (dnp no)
     (property "Reference" "C302" (at 128.27 165.1 0)
@@
     )
   )
-  (symbol (lib_id "_SCHLIB_HotPlate:CAP_100nF_6V3_X7R_C0201") (at 209.55 213.36 270) (unit 1)
+  (symbol (lib_id "_SCHLIB_HotPlate:CAP_CER_100nF_6V3_X7R_C0201") (at 209.55 213.36 270) (unit 1)
     (in_bom yes) (on_board yes) (dnp no)
     (property "Reference" "C308" (at 212.09 214.63 90)
@@
     )
   )
-  (symbol (lib_id "_SCHLIB_HotPlate:CAP_10uF_16V_X5R_C0603") (at 186.69 213.36 270) (unit 1)
+  (symbol (lib_id "_SCHLIB_HotPlate:CAP_CER_10uF_16V_X5R_C0603") (at 186.69 213.36 270) (unit 1)
     (in_bom yes) (on_board yes) (dnp no)
     (property "Reference" "C307" (at 189.23 214.63 90)
@@
     )
   )
-  (symbol (lib_id "_SCHLIB_HotPlate:CAP_100nF_6V3_X7R_C0201") (at 430.53 219.71 270) (unit 1)
+  (symbol (lib_id "_SCHLIB_HotPlate:CAP_CER_100nF_6V3_X7R_C0201") (at 430.53 219.71 270) (unit 1)
     (in_bom yes) (on_board yes) (dnp no)
     (property "Reference" "C311" (at 433.07 220.98 90)
@@
     )
   )
-  (symbol (lib_id "_SCHLIB_HotPlate:CAP_10uF_16V_X5R_C0603") (at 87.63 208.28 270) (unit 1)
+  (symbol (lib_id "_SCHLIB_HotPlate:CAP_CER_10uF_16V_X5R_C0603") (at 87.63 208.28 270) (unit 1)
     (in_bom yes) (on_board yes) (dnp no)
     (property "Reference" "C305" (at 90.17 209.55 90)
@@
     )
   )
-  (symbol (lib_id "_SCHLIB_HotPlate:CAP_100nF_6V3_X7R_C0201") (at 110.49 208.28 270) (unit 1)
+  (symbol (lib_id "_SCHLIB_HotPlate:CAP_CER_100nF_6V3_X7R_C0201") (at 110.49 208.28 270) (unit 1)
     (in_bom yes) (on_board yes) (dnp no)
     (property "Reference" "C306" (at 113.03 209.55 90)
@@
     )
   )
-  (symbol (lib_id "_SCHLIB_HotPlate:CAP_100nF_6V3_X7R_C0201") (at 346.71 213.36 270) (unit 1)
+  (symbol (lib_id "_SCHLIB_HotPlate:CAP_CER_100nF_6V3_X7R_C0201") (at 346.71 213.36 270) (unit 1)
     (in_bom yes) (on_board yes) (dnp no)
     (property "Reference" "C309" (at 349.25 214.63 90)
@@
     )
   )
-  (symbol (lib_id "_SCHLIB_HotPlate:CAP_12pF_50V_C0G_C0201") (at 125.73 148.59 180) (unit 1)
+  (symbol (lib_id "_SCHLIB_HotPlate:CAP_CER_12pF_50V_C0G_C0201") (at 125.73 148.59 180) (unit 1)
     (in_bom yes) (on_board yes) (dnp no)
     (property "Reference" "C301" (at 128.27 147.32 0)
@@
     )
   )
-  (symbol (lib_id "_SCHLIB_HotPlate:CAP_100nF_6V3_X7R_C0201") (at 68.58 185.42 270) (unit 1)
+  (symbol (lib_id "_SCHLIB_HotPlate:CAP_CER_100nF_6V3_X7R_C0201") (at 68.58 185.42 270) (unit 1)
     (in_bom yes) (on_board yes) (dnp no)
     (property "Reference" "C304" (at 71.12 187.96 90)
@@
     )
   )
-  (symbol (lib_id "_SCHLIB_HotPlate:CAP_100nF_6V3_X7R_C0201") (at 430.53 181.61 270) (unit 1)
+  (symbol (lib_id "_SCHLIB_HotPlate:CAP_CER_100nF_6V3_X7R_C0201") (at 430.53 181.61 270) (unit 1)
     (in_bom yes) (on_board yes) (dnp no)
     (property "Reference" "C303" (at 433.07 182.88 90)
@@
     )
   )
-  (symbol (lib_id "_SCHLIB_HotPlate:CAP_10uF_16V_X5R_C0603") (at 370.84 213.36 270) (unit 1)
+  (symbol (lib_id "_SCHLIB_HotPlate:CAP_CER_10uF_16V_X5R_C0603") (at 370.84 213.36 270) (unit 1)
     (in_bom yes) (on_board yes) (dnp no)
     (property "Reference" "C310" (at 373.38 214.63 90)
