File: Hardware/v1_20230725/Design Folder/_HW_HotPlate/[04] - THERMOCOUPLE DRIVER.kicad_sch (KiCad schematic)
At the start: 10 parts, among them J401 RECEPT_2X1_VERT_2.54MM, U401 MAX31855JASA+T

Commit message: Library updated
Parts:
- C401: symbol _SCHLIB_HotPlate:CAP_10nF_6V3_X7R_C0201 -> _SCHLIB_HotPlate:CAP_CER_10nF_6V3_X7R_C0201
- C402: symbol _SCHLIB_HotPlate:CAP_10uF_16V_X5R_C0603 -> _SCHLIB_HotPlate:CAP_CER_10uF_16V_X5R_C0603
- C403: symbol _SCHLIB_HotPlate:CAP_100nF_6V3_X7R_C0201 -> _SCHLIB_HotPlate:CAP_CER_100nF_6V3_X7R_C0201
Changed lines of the file:
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@@
     )
   )
-  (symbol (lib_id "_SCHLIB_HotPlate:CAP_10nF_6V3_X7R_C0201") (at 214.63 158.75 270) (unit 1)
+  (symbol (lib_id "_SCHLIB_HotPlate:CAP_CER_10nF_6V3_X7R_C0201") (at 214.63 158.75 270) (unit 1)
     (in_bom yes) (on_board yes) (dnp no)
     (property "Reference" "C401" (at 217.17 160.02 90)
@@
     )
   )
-  (symbol (lib_id "_SCHLIB_HotPlate:CAP_10uF_16V_X5R_C0603") (at 214.63 177.8 270) (unit 1)
+  (symbol (lib_id "_SCHLIB_HotPlate:CAP_CER_10uF_16V_X5R_C0603") (at 214.63 177.8 270) (unit 1)
     (in_bom yes) (on_board yes) (dnp no)
     (property "Reference" "C402" (at 217.17 179.07 90)
@@
     )
   )
-  (symbol (lib_id "_SCHLIB_HotPlate:CAP_100nF_6V3_X7R_C0201") (at 236.22 177.8 270) (unit 1)
+  (symbol (lib_id "_SCHLIB_HotPlate:CAP_CER_100nF_6V3_X7R_C0201") (at 236.22 177.8 270) (unit 1)
     (in_bom yes) (on_board yes) (dnp no)
     (property "Reference" "C403" (at 238.76 179.07 90)
