File: Hardware/v1_20230725/Design Folder/_HW_HotPlate/[06] - GLCD 84X48 Driver.kicad_sch (KiCad schematic)
At the start: 10 parts, among them J601 RECEPT_4X2_RA_2.54MM

Commit message: Library updated
Parts:
- C601: symbol _SCHLIB_HotPlate:CAP_10uF_16V_X5R_C0603 -> _SCHLIB_HotPlate:CAP_CER_10uF_16V_X5R_C0603
- C602: symbol _SCHLIB_HotPlate:CAP_100nF_6V3_X7R_C0201 -> _SCHLIB_HotPlate:CAP_CER_100nF_6V3_X7R_C0201
Changed lines of the file:
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@@
     )
   )
-  (symbol (lib_id "_SCHLIB_HotPlate:CAP_10uF_16V_X5R_C0603") (at 198.12 133.35 270) (unit 1)
+  (symbol (lib_id "_SCHLIB_HotPlate:CAP_CER_10uF_16V_X5R_C0603") (at 198.12 133.35 270) (unit 1)
     (in_bom yes) (on_board yes) (dnp no)
     (property "Reference" "C601" (at 200.66 134.62 90)
@@
     )
   )
-  (symbol (lib_id "_SCHLIB_HotPlate:CAP_100nF_6V3_X7R_C0201") (at 381 161.29 270) (unit 1)
+  (symbol (lib_id "_SCHLIB_HotPlate:CAP_CER_100nF_6V3_X7R_C0201") (at 381 161.29 270) (unit 1)
     (in_bom yes) (on_board yes) (dnp no)
     (property "Reference" "C602" (at 383.54 162.56 90)
