File: Hardware/v1_20230725/Design Folder/_HW_HotPlate/[07] - Rotary Encoder + PB Driver.kicad_sch (KiCad schematic)
At the start: 15 parts, among them J701 RECEPT_5X1_RA_2.54MM, U701 SN74LVC1G17DBVR, U702 SN74LVC1G17DBVR, U703 DLPT05A-7_5V_17A, U704 SN74LVC1G17DBVR

Commit message: Library updated
Parts:
- C701, C702, C704: symbol _SCHLIB_HotPlate:CAP_10uF_16V_X5R_C0603 -> _SCHLIB_HotPlate:CAP_CER_10uF_16V_X5R_C0603
- C703: symbol _SCHLIB_HotPlate:CAP_100nF_6V3_X7R_C0201 -> _SCHLIB_HotPlate:CAP_CER_100nF_6V3_X7R_C0201
Changed lines of the file:
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@@
     )
   )
-  (symbol (lib_id "_SCHLIB_HotPlate:CAP_100nF_6V3_X7R_C0201") (at 187.96 195.58 270) (unit 1)
+  (symbol (lib_id "_SCHLIB_HotPlate:CAP_CER_100nF_6V3_X7R_C0201") (at 187.96 195.58 270) (unit 1)
     (in_bom yes) (on_board yes) (dnp no)
     (property "Reference" "C703" (at 190.5 196.85 90)
@@
     )
   )
-  (symbol (lib_id "_SCHLIB_HotPlate:CAP_10uF_16V_X5R_C0603") (at 283.21 245.11 270) (unit 1)
+  (symbol (lib_id "_SCHLIB_HotPlate:CAP_CER_10uF_16V_X5R_C0603") (at 283.21 245.11 270) (unit 1)
     (in_bom yes) (on_board yes) (dnp no)
     (property "Reference" "C704" (at 285.75 246.38 90)
@@
     )
   )
-  (symbol (lib_id "_SCHLIB_HotPlate:CAP_10uF_16V_X5R_C0603") (at 281.94 173.99 270) (unit 1)
+  (symbol (lib_id "_SCHLIB_HotPlate:CAP_CER_10uF_16V_X5R_C0603") (at 281.94 173.99 270) (unit 1)
     (in_bom yes) (on_board yes) (dnp no)
     (property "Reference" "C702" (at 284.48 175.26 90)
@@
     )
   )
-  (symbol (lib_id "_SCHLIB_HotPlate:CAP_10uF_16V_X5R_C0603") (at 283.21 133.35 270) (unit 1)
+  (symbol (lib_id "_SCHLIB_HotPlate:CAP_CER_10uF_16V_X5R_C0603") (at 283.21 133.35 270) (unit 1)
     (in_bom yes) (on_board yes) (dnp no)
     (property "Reference" "C701" (at 285.75 134.62 90)
