File: Hardware/v1_20230725/Design Folder/_HW_HotPlate/[11] - POWER SUPPLY.kicad_sch (KiCad schematic)
At the start: 28 parts, among them U1101 MIC5528-3.3YMT-TR, U1102 MIC5528-3.3YMT-TR

Commit message: Library updated
Parts:
- C1101: symbol _SCHLIB_HotPlate:CAP_100nF_50V_X7R_C0603 -> _SCHLIB_HotPlate:CAP_CER_100nF_50V_X7R_C0603
- C1102: symbol _SCHLIB_HotPlate:CAP_1nF_450V_C0G_C0805 -> _SCHLIB_HotPlate:CAP_CER_1nF_450V_C0G_C0805
- C1103, C1104, C1105, C1106: symbol _SCHLIB_HotPlate:CAP_10uF_16V_X5R_C0603 -> _SCHLIB_HotPlate:CAP_CER_10uF_16V_X5R_C0603
Changed lines of the file:
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@@
     (effects (font (size 1.27 1.27)) (justify left))
   )
-  (symbol (lib_id "_SCHLIB_HotPlate:CAP_10uF_16V_X5R_C0603") (at 153.67 261.62 270) (unit 1)
+  (symbol (lib_id "_SCHLIB_HotPlate:CAP_CER_10uF_16V_X5R_C0603") (at 153.67 261.62 270) (unit 1)
     (in_bom yes) (on_board yes) (dnp no)
     (property "Reference" "C1105" (at 156.21 262.89 90)
@@
     )
   )
-  (symbol (lib_id "_SCHLIB_HotPlate:CAP_100nF_50V_X7R_C0603") (at 412.75 130.81 270) (unit 1)
+  (symbol (lib_id "_SCHLIB_HotPlate:CAP_CER_100nF_50V_X7R_C0603") (at 412.75 130.81 270) (unit 1)
     (in_bom yes) (on_board yes) (dnp no)
     (property "Reference" "C1101" (at 415.29 132.08 90)
@@
     )
   )
-  (symbol (lib_id "_SCHLIB_HotPlate:CAP_10uF_16V_X5R_C0603") (at 302.26 208.28 270) (unit 1)
+  (symbol (lib_id "_SCHLIB_HotPlate:CAP_CER_10uF_16V_X5R_C0603") (at 302.26 208.28 270) (unit 1)
     (in_bom yes) (on_board yes) (dnp no)
     (property "Reference" "C1104" (at 304.8 209.55 90)
@@
     )
   )
-  (symbol (lib_id "_SCHLIB_HotPlate:CAP_10uF_16V_X5R_C0603") (at 302.26 269.24 270) (unit 1)
+  (symbol (lib_id "_SCHLIB_HotPlate:CAP_CER_10uF_16V_X5R_C0603") (at 302.26 269.24 270) (unit 1)
     (in_bom yes) (on_board yes) (dnp no)
     (property "Reference" "C1106" (at 304.8 270.51 90)
@@
     )
   )
-  (symbol (lib_id "_SCHLIB_HotPlate:CAP_10uF_16V_X5R_C0603") (at 153.67 200.66 270) (unit 1)
+  (symbol (lib_id "_SCHLIB_HotPlate:CAP_CER_10uF_16V_X5R_C0603") (at 153.67 200.66 270) (unit 1)
     (in_bom yes) (on_board yes) (dnp no)
     (property "Reference" "C1103" (at 156.21 201.93 90)
@@
     )
   )
-  (symbol (lib_id "_SCHLIB_HotPlate:CAP_1nF_450V_C0G_C0805") (at 274.32 154.94 180) (unit 1)
+  (symbol (lib_id "_SCHLIB_HotPlate:CAP_CER_1nF_450V_C0G_C0805") (at 274.32 154.94 180) (unit 1)
     (in_bom yes) (on_board yes) (dnp no)
     (property "Reference" "C1102" (at 276.86 153.67 0)
